File: Leds.kicad_sch (KiCad schematic)
At the start: 16 parts, among them Q2 NTK3134N, Q3 NTK3134N, SW1 EVQP7A01P, SW2 EVQP7A01P

Commit message: fix(hardware): replace jumper/passive footprints with 0402 and refine schematics
- Replace 0-ohm jumper resistors with 0402 package equivalents
- Reduce package size on several capacitors
- Correct and simplify several schematic symbols (replaced with
  simplified equivalents where the original was overcomplicated)
- Bump lib submodule to the updated component library (renamed
  switch footprints, new Conn_01x02_MountingPin symbol, pad/pin
  numbering fixes, approved IPN assignments, Workart artwork library)
- Register Workart.pretty in fp-lib-table
- Mark J3 as DNP in mcu.kicad_sch
- Continue schematic wiring/placement (Leds.kicad_sch, tessera.kicad_sch)
  and PCB routing/placement (tessera.kicad_pcb)
- Add board outline source (Images/pcb_size.dxf, pcb_shape.FCStd) and
  silkscreen artwork sources (Logos/) for the Workart footprints
- Complete preliminary version of PCB
Parts:
- SW1, SW2: footprint Button_Switch:Panasonic_EVQP7K_EVQP7A -> Button_Switch:Panasonic_switch_EVQP7K_EVQP7A
Connections:
- net GND: now also D1.1 (K); no longer R31.2
- net RST_PB: now also R36.2
- net USR_PB: now also R37.2
- net VCC_LED_RF: now also R31.1; no longer D1.2 (A)
- new net: D1.2 (A), R31.2
Other:
- moved on the sheet: R31, R36, R37, TP17, TP18
