File: USB_Conn.kicad_sch (KiCad schematic)
At the start: 6 parts, among them J1 USB-C, U1 USBLC6-2P6

Commit message: fix(hardware): replace jumper/passive footprints with 0402 and refine schematics
- Replace 0-ohm jumper resistors with 0402 package equivalents
- Reduce package size on several capacitors
- Correct and simplify several schematic symbols (replaced with
  simplified equivalents where the original was overcomplicated)
- Bump lib submodule to the updated component library (renamed
  switch footprints, new Conn_01x02_MountingPin symbol, pad/pin
  numbering fixes, approved IPN assignments, Workart artwork library)
- Register Workart.pretty in fp-lib-table
- Mark J3 as DNP in mcu.kicad_sch
- Continue schematic wiring/placement (Leds.kicad_sch, tessera.kicad_sch)
  and PCB routing/placement (tessera.kicad_pcb)
- Add board outline source (Images/pcb_size.dxf, pcb_shape.FCStd) and
  silkscreen artwork sources (Logos/) for the Workart footprints
- Complete preliminary version of PCB
Connections:
- net GND: now also J1.S2 (SHIELD), J1.S3 (SHIELD), J1.S4 (SHIELD)
- net USB_D+: now reaches J1.A6 (D+), J1.B6 (D+), U1.3 (I/O2)
- net USB_D-: now reaches J1.A7 (D-), J1.B7 (D-), U1.1 (I/O1)
Changed lines of the file:
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@@
+		)
+	)
+	(label "USB_D+"
+		(at 135.89 81.28 0)
+		(fields_autoplaced yes)
+		(effects
+			(font
+				(size 1.27 1.27)
+			)
+			(justify left bottom)
+		)
+	)
+	(label "USB_D-"
+		(at 135.89 78.74 0)
+		(fields_autoplaced yes)
+		(effects
+			(font
+				(size 1.27 1.27)
+			)
+			(justify left bottom)
 		)
 	)
@@
 		(pin "B8"
 		)
+		(pin "S4"
+		)
+		(pin "S2"
+		)
+		(pin "S3"
+		)
 		(instances
