File: nfc.kicad_sch (KiCad schematic)
At the start: 14 parts, among them U6 ST25DV64KC-JF6D3

Commit message: fix(hardware): mirror secure element power switch
- Mirror Q1
- Change R42 to pull-down
- Fix some overlapping graphics
Parts:
- AE1: now left out of the parts list
Changed lines of the file:
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@@
 	(title_block
 		(title "NFC Interface")
-		(date "2026-10-11")
+		(date "2026-10-26")
 	)
 	(junction
@@
 		(unit 1)
 		(exclude_from_sim no)
-		(in_bom yes)
+		(in_bom no)
 		(on_board yes)
 		(dnp no)
