File: power.kicad_sch (KiCad schematic)
At the start: 25 parts, among them J2 532610271, Q1 NTK3139P, U2 BQ25170J, U3 TPS62840DLCR

Commit message: fix(hardware): mirror secure element power switch
- Mirror Q1
- Change R42 to pull-down
- Fix some overlapping graphics
Connections:
- net 3V: now also Q1.2 (S); no longer Q1.3 (D)
- net 3V_SEC: now also Q1.3 (D); no longer Q1.2 (S)
Other:
- moved on the sheet: Q1
Changed lines of the file:
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@@
 	(title_block
 		(title "Power Supply")
-		(date "2026-10-11")
+		(date "2026-10-26")
 	)
 	(junction
@@
 	(symbol
 		(lib_id "catalog:Transistors/NTK3139P")
-		(at 223.52 115.57 90)
+		(at 223.52 115.57 270)
+		(mirror x)
 		(unit 1)
 		(exclude_from_sim no)
@@
 		)
 		(property "Footprint" "Packages_TO_SOT:SOT-723"
-			(at 220.98 110.49 0)
+			(at 226.06 110.49 0)
 			(effects
 				(font
