File: stsafe120.kicad_sch (KiCad schematic)
At the start: 5 parts, among them U7 STSAFA120DFSPL05

Commit message: fix(hardware): mirror secure element power switch
- Mirror Q1
- Change R42 to pull-down
- Fix some overlapping graphics
Connections:
- net GND: now also R42.2
- net /RST: now also R42.1; no longer R42.2
- net at C18.1, R41.1, U7.2 (VCC): no longer R42.1
Other:
- moved on the sheet: R42
