File: tessera.kicad_pcb (KiCad board)
At the start: 4 copper layers, 54 x 85.6 mm, 113 parts, among them J1 USB-C, J2 532610271, J3 PinHeader_2x05, Q1 NTK3139P, Q2 NTK3134N, Q3 NTK3134N, SW1 EVQP7A01P, SW2 EVQP7A01P, U1 USBLC6-2P6, U2 BQ25170J, U3 TPS62840DLCR, U4 ISP1807-LR-RS, U5 D3V3XA4B10LP, U6 ST25DV64KC-JF6D3, U7 STSAFA120DFSPL05

Commit message: fix(hardware): mirror secure element power switch
- Mirror Q1
- Change R42 to pull-down
- Fix some overlapping graphics
Parts:
- turned Q1 to 90 degrees
- turned R42 to -90 degrees
Connections:
- Q1 pad 2: VCC_SEC -> VCC
- Q1 pad 3: VCC -> VCC_SEC
- R42 pad 1: Net-(U7-VCC) -> /Project Architecture/SEC_RST
- R42 pad 2: /Project Architecture/SEC_RST -> GND
Routing:
- net Net-(U7-VCC): track 5.18 -> 2.29 mm
- net VCC: track 166.7 -> 165.5 mm
- net /Project Architecture/SEC_PW_CTRL: track 14.1 -> 13.5 mm
